File: 18650_1S3P/18650_1S3P.sch (EAGLE design)
At the start: 31 parts, among them Q1 DMG3404, Q2 DMG3404, Q3 DMG3404

Commit message: Updated diode part number, new BoM
Fixed diode part number to be correct SOD323 diode instead of SOD523 diode, regenerated BoM to reflect change
Parts:
- D4, D5, D6: DIGIKEY 1N4148WTDICT-ND -> 1N4148WS-FDICT-ND; MPN 1N4148WT-7 -> 1N4148WS-7-F
Changed lines of the file:
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@@
 <?xml version="1.0" encoding="utf-8"?>
 <!DOCTYPE eagle SYSTEM "eagle.dtd">
-<eagle version="9.4.2">
+<eagle version="9.6.2">
 <drawing>
 <settings>
@@
 <part name="R7" library="bschulz_passives" deviceset="R-EU_" device="R0603" technology="100K" value="100k"/>
 <part name="D4" library="bschulz" deviceset="DIODE" device="SOD-323" value="1N4148">
-<attribute name="DIGIKEY" value="1N4148WTDICT-ND"/>
+<attribute name="DIGIKEY" value="1N4148WS-FDICT-ND"/>
 <attribute name="MF" value="Diodes Inc"/>
-<attribute name="MPN" value="1N4148WT-7"/>
+<attribute name="MPN" value="1N4148WS-7-F"/>
 </part>
 <part name="D5" library="bschulz" deviceset="DIODE" device="SOD-323" value="1N4148">
-<attribute name="DIGIKEY" value="1N4148WTDICT-ND"/>
+<attribute name="DIGIKEY" value="1N4148WS-FDICT-ND"/>
 <attribute name="MF" value="Diodes Inc"/>
-<attribute name="MPN" value="1N4148WT-7"/>
+<attribute name="MPN" value="1N4148WS-7-F"/>
 </part>
 <part name="D6" library="bschulz" deviceset="DIODE" device="SOD-323" value="1N4148">
-<attribute name="DIGIKEY" value="1N4148WTDICT-ND"/>
+<attribute name="DIGIKEY" value="1N4148WS-FDICT-ND"/>
 <attribute name="MF" value="Diodes Inc"/>
-<attribute name="MPN" value="1N4148WT-7"/>
+<attribute name="MPN" value="1N4148WS-7-F"/>
 </part>
 </parts>
