File: 18650_1S3P/Hardware/18650_1S3P_Smart_VertCon.sch (EAGLE design)
At the start: 75 parts, among them J1 CONN_3MICROFIT_RT, J2 GEMS_POWER_PLUGOUTPUT, Q1 AON7522E, Q2 AON7522E, Q3 AON7522E, Q4 AON7522E, Q5 AON7522E, Q6 AON7522E, Q7 DMP2008, Q8 DMP2008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

Commit message: Added 18650_1S3P_Smart v1.2 (very and normal)
Added v1.2 updates for both systems
Parts:
- BT1, BT2, BT3: DIGIKEY (none) -> 36-1042-ND; MPN (none) -> 1042
Changed lines of the file:
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@@
 <part name="Q1" library="bschulz" deviceset="MOSFET-NCH" device="-AON7522E" value="AON7522E"/>
 <part name="Q2" library="bschulz" deviceset="MOSFET-NCH" device="-AON7522E" value="AON7522E"/>
-<part name="BT1" library="bschulz" deviceset="18650" device="1042P_NOSILK" value="186501042P_NOSILK"/>
+<part name="BT1" library="bschulz" deviceset="18650" device="1042P_NOSILK" value="186501042P_NOSILK">
+<attribute name="DIGIKEY" value="36-1042-ND"/>
+<attribute name="MPN" value="1042"/>
+</part>
 <part name="D1" library="bschulz" deviceset="DIODE_SCHOTTKY" device="SOD-323">
 <attribute name="DIGIKEY" value="BAT54WS-FDICT-ND"/>
@@
 <part name="Q3" library="bschulz" deviceset="MOSFET-NCH" device="-AON7522E" value="AON7522E"/>
 <part name="Q4" library="bschulz" deviceset="MOSFET-NCH" device="-AON7522E" value="AON7522E"/>
-<part name="BT2" library="bschulz" deviceset="18650" device="1042P_NOSILK" value="186501042P_NOSILK"/>
+<part name="BT2" library="bschulz" deviceset="18650" device="1042P_NOSILK" value="186501042P_NOSILK">
+<attribute name="DIGIKEY" value="36-1042-ND"/>
+<attribute name="MPN" value="1042"/>
+</part>
 <part name="D2" library="bschulz" deviceset="DIODE_SCHOTTKY" device="SOD-323">
 <attribute name="DIGIKEY" value="BAT54WS-FDICT-ND"/>
@@
 <part name="Q5" library="bschulz" deviceset="MOSFET-NCH" device="-AON7522E" value="AON7522E"/>
 <part name="Q6" library="bschulz" deviceset="MOSFET-NCH" device="-AON7522E" value="AON7522E"/>
-<part name="BT3" library="bschulz" deviceset="18650" device="1042P_NOSILK" value="186501042P_NOSILK"/>
+<part name="BT3" library="bschulz" deviceset="18650" device="1042P_NOSILK" value="186501042P_NOSILK">
+<attribute name="DIGIKEY" value="36-1042-ND"/>
+<attribute name="MPN" value="1042"/>
+</part>
 <part name="D3" library="bschulz" deviceset="DIODE_SCHOTTKY" device="SOD-323">
 <attribute name="DIGIKEY" value="BAT54WS-FDICT-ND"/>
@@
 <instance part="J2" gate="G$1" x="167.64" y="182.88" smashed="yes">
 <attribute name="NAME" x="167.64" y="176.276" size="1.778" layer="95" ratio="15" align="center"/>
-<attribute name="DISP" x="167.64" y="188.468" size="2.54" layer="94" ratio="15" align="bottom-center"/>
 </instance>
 <instance part="R32" gate="G$1" x="195.58" y="180.34" smashed="yes" rot="R180">

Commit message: Changed folder structure to include legacy aspects
Also changed 1042P to 1042 to match manufactured version
Parts:
- BT1, BT2, BT3: value 186501042P_NOSILK -> 186501042; device bschulz:186501042P_NOSILK -> bschulz:186501042
Changed lines of the file:
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@@
 <layer number="128" name="_bValues" color="7" fill="1" visible="no" active="yes"/>
 <layer number="129" name="Mask" color="7" fill="1" visible="no" active="yes"/>
+<layer number="130" name="SMDSTROOK" color="7" fill="1" visible="no" active="no"/>
 <layer number="131" name="tAdjust" color="7" fill="1" visible="no" active="yes"/>
 <layer number="132" name="bAdjust" color="7" fill="1" visible="no" active="yes"/>
+<layer number="133" name="bottom_silk" color="7" fill="1" visible="no" active="no"/>
+<layer number="134" name="mbFinish" color="7" fill="1" visible="no" active="no"/>
+<layer number="135" name="mtGlue" color="7" fill="1" visible="no" active="no"/>
+<layer number="136" name="mbGlue" color="7" fill="1" visible="no" active="no"/>
+<layer number="137" name="mtTest" color="7" fill="1" visible="no" active="no"/>
+<layer number="138" name="mbTest" color="7" fill="1" visible="no" active="no"/>
+<layer number="139" name="mtKeepout" color="7" fill="1" visible="no" active="no"/>
+<layer number="140" name="mbKeepout" color="7" fill="1" visible="no" active="no"/>
+<layer number="141" name="mtRestrict" color="7" fill="1" visible="no" active="no"/>
+<layer number="142" name="mbRestrict" color="7" fill="1" visible="no" active="no"/>
+<layer number="143" name="mvRestrict" color="7" fill="1" visible="no" active="no"/>
 <layer number="144" name="Drill_legend" color="7" fill="1" visible="no" active="yes"/>
+<layer number="145" name="mHoles" color="7" fill="1" visible="no" active="no"/>
+<layer number="146" name="mMilling" color="7" fill="1" visible="no" active="no"/>
+<layer number="147" name="mMeasures" color="7" fill="1" visible="no" active="no"/>
+<layer number="148" name="mDocument" color="7" fill="1" visible="no" active="no"/>
+<layer number="149" name="mReference" color="7" fill="1" visible="no" active="no"/>
 <layer number="150" name="Notes" color="7" fill="1" visible="no" active="yes"/>
 <layer number="151" name="HeatSink" color="7" fill="1" visible="no" active="yes"/>
@@
 <layer number="154" name="FabDoc2" color="7" fill="1" visible="no" active="yes"/>
 <layer number="155" name="FabDoc3" color="7" fill="1" visible="no" active="yes"/>
+<layer number="166" name="AntennaArea" color="7" fill="1" visible="no" active="no"/>
+<layer number="168" name="4mmHeightArea" color="7" fill="1" visible="no" active="no"/>
+<layer number="191" name="mNets" color="7" fill="1" visible="no" active="no"/>
+<layer number="192" name="mBusses" color="7" fill="1" visible="no" active="no"/>
+<layer number="193" name="mPins" color="7" fill="1" visible="no" active="no"/>
+<layer number="194" name="mSymbols" color="7" fill="1" visible="no" active="no"/>
+<layer number="195" name="mNames" color="7" fill="1" visible="no" active="no"/>
+<layer number="196" name="mValues" color="7" fill="1" visible="no" active="no"/>
 <layer number="199" name="Contour" color="7" fill="1" visible="no" active="yes"/>
 <layer number="200" name="200bmp" color="7" fill="1" visible="no" active="yes"/>
@@
 <part name="Q1" library="bschulz" deviceset="MOSFET-NCH" device="-AON7522E" value="AON7522E"/>
 <part name="Q2" library="bschulz" deviceset="MOSFET-NCH" device="-AON7522E" value="AON7522E"/>
-<part name="BT1" library="bschulz" deviceset="18650" device="1042P_NOSILK" value="186501042P_NOSILK">
+<part name="BT1" library="bschulz" deviceset="18650" device="1042" value="186501042">
 <attribute name="DIGIKEY" value="36-1042-ND"/>
 <attribute name="MPN" value="1042"/>
@@
 <part name="Q3" library="bschulz" deviceset="MOSFET-NCH" device="-AON7522E" value="AON7522E"/>
 <part name="Q4" library="bschulz" deviceset="MOSFET-NCH" device="-AON7522E" value="AON7522E"/>
-<part name="BT2" library="bschulz" deviceset="18650" device="1042P_NOSILK" value="186501042P_NOSILK">
+<part name="BT2" library="bschulz" deviceset="18650" device="1042" value="186501042">
 <attribute name="DIGIKEY" value="36-1042-ND"/>
 <attribute name="MPN" value="1042"/>
@@
 <part name="Q5" library="bschulz" deviceset="MOSFET-NCH" device="-AON7522E" value="AON7522E"/>
 <part name="Q6" library="bschulz" deviceset="MOSFET-NCH" device="-AON7522E" value="AON7522E"/>
-<part name="BT3" library="bschulz" deviceset="18650" device="1042P_NOSILK" value="186501042P_NOSILK">
+<part name="BT3" library="bschulz" deviceset="18650" device="1042" value="186501042">
 <attribute name="DIGIKEY" value="36-1042-ND"/>
 <attribute name="MPN" value="1042"/>
